File: UccMicroDuino/UccMicroDuino.kicad_sch (KiCad schematic)
At the start: 8 parts, among them J2 Conn_01x10_Socket, J2 USB_A, U2 ATtiny85-20S

Commit message: Add files via upload
Parts:
- added D4: 3.6V 1/2mW, Diode_SMD:D_SOD-123, symbol Device:D_Zener
- added D5: LED, ledSmd:ledSMD, symbol Device:LED
- added R2, R3: 330Ω 5% 1/8W, Resistor_SMD:R_0805_2012Metric_Pad1.20x1.40mm_HandSolder, symbol Device:R
- added R4, R5: 68Ω 5% 1/8W, Resistor_SMD:R_0805_2012Metric_Pad1.20x1.40mm_HandSolder, symbol Device:R
- D2: renamed from D1; value D_Zener -> 3.6V 1/2mW
- R1: value R -> 1.5KΩ 5% 1/8W
- renumbered D5 to D1, J2 to J1, U2 to U1
Connections:
- net +5V: now also C1.1, D3.2 (A), J1.1 (Pin_1), U1.8 (VCC)
- net GND: now also C1.2, D2.2 (A), J1.2 (Pin_2), J2.4 (GND), U1.4 (GND), D4.2 (A), R2.2, R3.1
- net at D3.1 (K): now also R3.2
- net at R1.2: now also D2.1 (K), J2.2 (D-), R5.1
- net at U1.1 (~{RESET}/PB5): now also J1.9 (Pin_9)
- net at U1.2 (XTAL1/PB3): now also J1.7 (Pin_7), R5.2
- net at U1.3 (XTAL2/PB4): now also J1.8 (Pin_8), R4.1
- net at U1.5 (AREF/PB0): now also J1.4 (Pin_4)
- net at U1.6 (PB1): now also J1.5 (Pin_5), D5.2 (A)
- net at U1.7 (PB2): now also J1.6 (Pin_6)
- net at J2.1 (VBUS): now also D1.2 (A)
- net at J2.3 (D+): now also D4.1 (K), R4.2
- new net: D5.1 (K), R2.1
- no-connect marks 0 -> 2
Other:
- moved on the sheet: C1, D3, U1
