File: UccMicroDuino/UccMicroDuino.kicad_pcb (KiCad board)
At the start: 2 copper layers, 8 parts, among them J1 Conn_01x10_Socket, J2 USB_A, U1 ATtiny85-20S

Commit message: Add files via upload
Parts:
- added D4: 3.6V 1/2mW, Diode_SMD:D_SOD-123, F.Cu at (207.3, 66.0)
- added D5: LED, ledSmd:ledSMD, F.Cu at (190.0, 84.0)
- added R2: 330Ω 5% 1/8W, Resistor_SMD:R_0805_2012Metric_Pad1.20x1.40mm_HandSolder, F.Cu at (191.0, 78.0)
- added R3: 330Ω 5% 1/8W, Resistor_SMD:R_0805_2012Metric_Pad1.20x1.40mm_HandSolder, F.Cu at (182.0, 84.0)
- added R4: 68Ω 5% 1/8W, Resistor_SMD:R_0805_2012Metric_Pad1.20x1.40mm_HandSolder, F.Cu at (201.0, 70.0)
- added R5: 68Ω 5% 1/8W, Resistor_SMD:R_0805_2012Metric_Pad1.20x1.40mm_HandSolder, F.Cu at (198.0, 73.0)
- D2: value D_Zener -> 3.6V 1/2mW
- R1: value R -> 1.5KΩ 5% 1/8W
- moved D2 78.7 mm to (206.7, 76.0)
- moved U1 68.4 mm to (200.0, 86.0), turned to 180 degrees
- moved J1 64.7 mm to (183.8, 93.0), turned to 90 degrees
- moved C1 53.9 mm to (192.0, 75.0)
- moved R1 52.4 mm to (191.0, 69.0)
- moved D1 48.9 mm to (175.8, 71.0), turned to 180 degrees
- moved J2 47.0 mm to (177.0, 58.7), turned to -90 degrees
- moved D3 43.7 mm to (178.0, 77.0), turned to 90 degrees
Connections:
- C1 pad 1: unconnected-(C1-Pad1) -> +5V
- C1 pad 2: unconnected-(C1-Pad2) -> GND
- D1 pad 2: unconnected-(D1-A-Pad2) -> Net-(D1-A)
- D2 pad 1: unconnected-(D2-K-Pad1) -> Net-(D2-K)
- D2 pad 2: unconnected-(D2-A-Pad2) -> GND
- D3 pad 1: unconnected-(D3-K-Pad1) -> Net-(D3-K)
- D3 pad 2: unconnected-(D3-A-Pad2) -> +5V
- J1 pad 1: unconnected-(J1-Pin_1-Pad1) -> +5V
- J1 pad 2: unconnected-(J1-Pin_2-Pad2) -> GND
- J1 pad 4: unconnected-(J1-Pin_4-Pad4) -> Net-(J1-Pin_4)
- J1 pad 5: unconnected-(J1-Pin_5-Pad5) -> Net-(D5-A)
- J1 pad 6: unconnected-(J1-Pin_6-Pad6) -> Net-(J1-Pin_6)
- J1 pad 7: unconnected-(J1-Pin_7-Pad7) -> Net-(J1-Pin_7)
- J1 pad 8: unconnected-(J1-Pin_8-Pad8) -> Net-(J1-Pin_8)
- J1 pad 9: unconnected-(J1-Pin_9-Pad9) -> Net-(J1-Pin_9)
- J2 pad 1: unconnected-(J2-VBUS-Pad1) -> Net-(D1-A)
- J2 pad 2: unconnected-(J2-D--Pad2) -> Net-(D2-K)
- J2 pad 3: unconnected-(J2-D+-Pad3) -> Net-(D4-K)
- J2 pad 4: unconnected-(J2-GND-Pad4) -> GND
- R1 pad 2: unconnected-(R1-Pad2) -> Net-(D2-K)
- U1 pad 1: unconnected-(U1-~{RESET}/PB5-Pad1) -> Net-(J1-Pin_9)
- U1 pad 2: unconnected-(U1-XTAL1/PB3-Pad2) -> Net-(J1-Pin_7)
- U1 pad 3: unconnected-(U1-XTAL2/PB4-Pad3) -> Net-(J1-Pin_8)
- U1 pad 4: unconnected-(U1-GND-Pad4) -> GND
- U1 pad 5: unconnected-(U1-AREF/PB0-Pad5) -> Net-(J1-Pin_4)
- U1 pad 6: unconnected-(U1-PB1-Pad6) -> Net-(D5-A)
- U1 pad 7: unconnected-(U1-PB2-Pad7) -> Net-(J1-Pin_6)
- U1 pad 8: unconnected-(U1-VCC-Pad8) -> +5V
Routing:
- net GND: track 0.00 -> 129.3 mm
- net +5V: track 0.00 -> 66.6 mm
- net Net-(D4-K): track 0.00 -> 52.6 mm
- net Net-(D2-K): track 0.00 -> 48.9 mm
- net Net-(J1-Pin_8): track 0.00 -> 36.2 mm
- net Net-(J1-Pin_7): track 0.00 -> 25.2 mm
- net Net-(D5-A): track 0.00 -> 19.6 mm
- net Net-(D1-A): track 0.00 -> 15.7 mm
- net Net-(J1-Pin_4): track 0.00 -> 11.8 mm
- net Net-(J1-Pin_6): track 0.00 -> 8.00 mm
- net Net-(D5-K): track 0.00 -> 6.75 mm
- net Net-(D3-K): track 0.00 -> 6.44 mm
- net Net-(J1-Pin_9): track 0.00 -> 5.27 mm
Other:
- board outline added: 45 x 45 mm
